File: Electronics/board.sch (EAGLE design)
At the start: 9 parts

Commit message: Added electronics
Parts:
- removed IC1: (no value), SparkFun-AnalogIC:556
- added ISP1: AVRISP-6, adafruit:AVRISP-6
- added R2, R3: (no value), SparkFun-Passives:RESISTOR0805-RES
- added U1: TINY85-20-DIP, SparkFun-DigitalIC:ATTINY45TINY85-20-DIP
Connections:
- new net 5V: ISP1.VCC, R2.2, R3.2, U1.VCC
- new net N$3: ISP1.MOSI, JP1.2, R2.1, U1.PB0(MOSI)
- new net N$4: ISP1.MISO, JP2.2, R3.1, U1.PB1(MISO)
- new net N$7: ISP1.RST, U1.PB5(NRES)
- new net N$8: ISP1.SCK, U1.PB2(SCK/ADC1)
- net ESCSIG: now also U1.PB4(ADC2); no longer JP1.2
- net GND: now also ISP1.GND, JP1.1, JP2.1, U1.GND
- net SERVOSIG: now also U1.PB3(ADC3); no longer JP2.1
Other:
- moved on the sheet: JP1, JP2, SERVO
